Commit message: Added a readme file for calibrate_chest and made the urdf for chest camera more accurate

File: strands_description/urdf/scitos_chest_camera.xacro (robot description, xacro)
@@ -28,5 +28,5 @@
     <!-- Z height from calibrate_chest -->
     <axis xyz="0 0 1"/>
-    <origin rpy="0 0 0" xyz="0.12 0 0" />
+    <origin rpy="0 0 0" xyz="-0.01 0 0" />
     <limit effort="1000" velocity="1000" lower="0.5" upper="1.5"/>
     <parent link="base_link"/>

Commit message: Fixing broken robot model
Closes #50

File: strands_description/urdf/scitos_chest_camera.xacro (robot description, xacro)
@@ -7,6 +7,6 @@
        xmlns:xacro="http://ros.org/wiki/xacro">
   <!-- calibration data -->
-  <!-- <include filename="$(find scitos_description)/urdf/scitos_calibration.xacro" /> -->
-  <link name="base_link" />
+  <xacro:include filename="$(find scitos_description)/urdf/scitos.xacro" />
+  <!--<link name="base_link" />-->
   <!-- Connect base to chest_xtion_link -->
   <link name="chest_xtion_link">
