Commit message: Starting the state publisher in the chest namespace and having a /chest/robot_description and a /robot_description parameter.

File: strands_description/urdf/scitos_all_robot_model.xacro (robot description, xacro)
@@ -7,6 +7,5 @@
        xmlns:xacro="http://ros.org/wiki/xacro">
   <!-- calibration data -->
-  <!-- <xacro:include filename="$(find scitos_description)/urdf/scitos_calibration.xacro" /> -->
-  <link name="base_link" />
+  <xacro:include filename="$(find scitos_description)/urdf/scitos.xacro" />
   <!-- Connect base to chest_xtion_link -->
   <link name="chest_xtion_link">

Commit message: Adjusted chest camera x direction

File: strands_description/urdf/scitos_all_robot_model.xacro (robot description, xacro)
@@ -27,5 +27,5 @@
     <!-- Z height from calibrate_chest -->
     <axis xyz="0 0 1"/>
-    <origin rpy="0 0 0" xyz="-0.01 0 0" />
+    <origin rpy="0 0 0" xyz="0.0294 0 0" />
     <limit effort="1000" velocity="1000" lower="0.5" upper="1.5"/>
     <parent link="base_link"/>

File: strands_description/urdf/scitos_chest_camera.xacro (robot description, xacro)
@@ -28,5 +28,5 @@
     <!-- Z height from calibrate_chest -->
     <axis xyz="0 0 1"/>
-    <origin rpy="0 0 0" xyz="-0.01 0 0" />
+    <origin rpy="0 0 0" xyz="0.0294 0 0" />
     <limit effort="1000" velocity="1000" lower="0.5" upper="1.5"/>
     <parent link="base_link"/>
